Commit message: refactor: put the reported pose on the drive axle midpoint
Gazebo reports the model frame origin, which sat 80 mm behind the drive
axle, so an in-place turn swung it through a chord: 88 to 143 mm for
90 degrees, against a 30 mm waypoint tolerance. Wheel odometry reported
exactly 0.0 mm for the same turns because DiffDrive derives it from the
axle midpoint, so the two disagreed by construction, and the twist the
EKF fuses as base_link's velocity was really the axle's.

Shifts every model coordinate by 80 mm so the model origin is the axle
midpoint, and renames the body link to chassis_link.

The rename is not cosmetic. ApplyLinkWrench applies the suction at the
canonical link's ORIGIN, not at its centre of mass. That was invisible
while the two coincided; moving the origin onto the axle moved the
suction with it and dropped the rear caster from 73.33 N to exactly
0.00 N, with all 73.34 N transferred to the drive wheels. Keeping the
chassis origin at the body centre keeps the suction where it was.

Verified: all 21 contact load measurements reproduce the recorded
baseline to within 0.08 N, and a 90 degree turn now moves the reported
pose by 38 to 63 mm, which is the gravity sliding alone.

The guide gains the base_link definition and the reason for it.

Co-Authored-By: Claude Opus 5 <noreply@anthropic.com>

File: src/climbot_gazebo/models/climbot/climbot.urdf.xacro (robot description, xacro)
@@ -34,10 +34,11 @@
   <xacro:property name="caster_mass" value="$(arg caster_mass)"/>
   <xacro:property name="half_track" value="${$(arg wheel_separation) / 2.0}"/>
-  <!-- Link poses in the Gazebo model are relative to the model origin, while
-       URDF joints are relative to base_link, so the body centre is removed. -->
-  <xacro:property name="wheel_offset_x" value="${$(arg wheel_axle_x) - base_x}"/>
-  <xacro:property name="wheel_offset_z" value="${wheel_radius - base_z}"/>
-  <xacro:property name="caster_offset_x" value="${$(arg caster_x) - base_x}"/>
-  <xacro:property name="caster_offset_z" value="${caster_radius - base_z}"/>
+  <!-- base_link is the drive axle midpoint at the wall contact plane, the same
+       origin the Gazebo model uses, so link coordinates carry over unchanged
+       and the body is an offset on base_link rather than its origin. -->
+  <xacro:property name="wheel_offset_x" value="$(arg wheel_axle_x)"/>
+  <xacro:property name="wheel_offset_z" value="${wheel_radius}"/>
+  <xacro:property name="caster_offset_x" value="$(arg caster_x)"/>
+  <xacro:property name="caster_offset_z" value="${caster_radius}"/>
   <material name="body_blue">
     <color rgba="0.10 0.32 0.80 1"/>
@@ -77,5 +78,5 @@
       <parent link="base_link"/>
       <child link="${side}_wheel_link"/>
-      <origin xyz="${wheel_offset_x} ${sign * half_track - base_y} ${wheel_offset_z}"
+      <origin xyz="${wheel_offset_x} ${sign * half_track} ${wheel_offset_z}"
               rpy="1.57079632679 0 0"/>
       <!-- The roll above sends the wheel's local +Z along the model's -Y, so
@@ -86,4 +87,5 @@
   <link name="base_link">
     <inertial>
+      <origin xyz="${base_x} ${base_y} ${base_z}"/>
       <mass value="${base_mass}"/>
       <inertia
@@ -94,4 +96,5 @@
     </inertial>
     <visual>
+      <origin xyz="${base_x} ${base_y} ${base_z}"/>
       <geometry>
         <box size="${length} ${width} ${thickness}"/>
@@ -100,5 +103,6 @@
     </visual>
     <visual>
-      <origin xyz="${length / 2.0 - 0.03} 0 ${thickness / 2.0 + 0.011}"/>
+      <origin xyz="${base_x + length / 2.0 - 0.03} ${base_y}
+                   ${base_z + thickness / 2.0 + 0.011}"/>
       <geometry>
         <box size="0.07 ${width * 0.41} 0.025"/>
@@ -107,4 +111,5 @@
     </visual>
     <collision>
+      <origin xyz="${base_x} ${base_y} ${base_z}"/>
       <geometry>
         <box size="${length} ${width} ${thickness}"/>
@@ -112,6 +117,6 @@
     </collision>
   </link>
-  <!-- The IMU sits at the body origin, so this frame is coincident with
-       base_link. It exists so an offset mount only needs robot.yaml changed. -->
+  <!-- The IMU is co-located with base_link, so this frame is coincident
+       with it. It exists so an offset mount only needs robot.yaml changed. -->
   <link name="imu_link"/>
   <joint name="imu_joint" type="fixed">
@@ -147,5 +152,5 @@
     <parent link="base_link"/>
     <child link="caster_ball_link"/>
-    <origin xyz="${caster_offset_x} ${-base_y} ${caster_offset_z}" rpy="0 0 0"/>
+    <origin xyz="${caster_offset_x} 0 ${caster_offset_z}" rpy="0 0 0"/>
   </joint>
 </robot>

File: src/climbot_gazebo/models/climbot/model.sdf.xacro (robot description, xacro)
@@ -41,4 +41,7 @@
   <xacro:property name="thickness" value="$(arg base_thickness)"/>
   <xacro:property name="base_mass" value="$(arg base_mass)"/>
+  <xacro:property name="base_x" value="$(arg base_x)"/>
+  <xacro:property name="base_y" value="$(arg base_y)"/>
+  <xacro:property name="base_z" value="$(arg base_z)"/>
   <xacro:property name="wheel_radius" value="$(arg wheel_radius)"/>
   <xacro:property name="wheel_width" value="$(arg wheel_width)"/>
@@ -110,5 +113,5 @@
     </link>
     <joint name="${side}_wheel_joint" type="revolute">
-      <parent>base_link</parent>
+      <parent>chassis_link</parent>
       <child>${side}_wheel_link</child>
       <axis>
@@ -126,5 +129,5 @@
     </joint>
   </xacro:macro>
-  <model name="climbot" canonical_link="base_link">
+  <model name="climbot" canonical_link="chassis_link">
     <self_collide>false</self_collide>
     <!--
@@ -132,6 +135,15 @@
       the driving surface. The world rotates this model onto the wall.
     -->
-    <link name="base_link">
-      <pose>$(arg base_x) $(arg base_y) $(arg base_z) 0 0 0</pose>
+    <!--
+      The model origin is the drive axle midpoint at the wall contact plane, so
+      the pose Gazebo reports is the point a differential drive rotates about
+      and an in-place turn no longer swings it.
+      This chassis link keeps its origin at the body centre because
+      ApplyLinkWrench applies the suction at the canonical link's ORIGIN, not
+      at its centre of mass. Moving this origin moves the suction, and putting
+      it on the axle drops the rear caster to zero normal load.
+    -->
+    <link name="chassis_link">
+      <pose>${base_x} ${base_y} ${base_z} 0 0 0</pose>
       <inertial>
         <mass>${base_mass}</mass>
@@ -176,7 +188,6 @@
         </material>
       </visual>
-      <!-- The IMU is rigidly mounted at the body origin, so imu_link and
-           base_link differ only by the identity transform published by
-           robot_state_publisher. -->
+      <!-- Mounted on the chassis; the ROS-side frame is base_link, which
+           robot_state_publisher places at the model origin. -->
       <sensor name="imu" type="imu">
         <always_on>true</always_on>
@@ -248,5 +259,5 @@
     </link>
     <joint name="caster_ball_joint" type="ball">
-      <parent>base_link</parent>
+      <parent>chassis_link</parent>
       <child>caster_ball_link</child>
     </joint>
