Commit message: feat: add thirty-frame LED flat-field calibration

File: src/climbot_gazebo/models/climbot/model.sdf.xacro (robot description, xacro)
@@ -71,5 +71,5 @@
   <xacro:arg name="camera_far_clip" default="20.0"/>
   <xacro:arg name="camera_noise_mean" default="0.0"/>
-  <xacro:arg name="camera_noise_stddev" default="0.002"/>
+  <xacro:arg name="camera_noise_stddev" default="0.004"/>
   <xacro:arg name="camera_visualize" default="false"/>
   <xacro:arg name="inspection_led_x" default="0.380"/>

File: src/climbot_gazebo/worlds/climbot_wall.sdf.xacro (robot description, xacro)
@@ -22,4 +22,5 @@
   <xacro:arg name="spawn_yaw" default="1.5707963267948966"/>
   <xacro:arg name="inspection_target" default="false"/>
+  <xacro:arg name="inspection_flat_field_target" default="false"/>
   <xacro:arg name="target_lateral" default="0.34"/>
   <xacro:arg name="target_height" default="2.0"/>
@@ -235,4 +236,18 @@
           </visual>
         </xacro:if>
+        <!-- Uniform low-specular target used only to measure the LED/camera
+             flat field. It exceeds the full distorted footprint, so every
+             output pixel sees the same nominal reflectance. -->
+        <xacro:if value="$(arg inspection_flat_field_target)">
+          <visual name="inspection_flat_field_target">
+            <pose>${decal_x + 0.004} ${target_lateral} ${target_height - centre_z} 0 0 0</pose>
+            <geometry><box><size>0.004 0.42 0.68</size></box></geometry>
+            <material>
+              <ambient>0.50 0.50 0.50 1</ambient>
+              <diffuse>0.50 0.50 0.50 1</diffuse>
+              <specular>0.01 0.01 0.01 1</specular>
+            </material>
+          </visual>
+        </xacro:if>
       </link>
     </model>

Commit message: feat(inspection): harden moonlit capture runtime

File: src/climbot_gazebo/models/climbot/model.sdf.xacro (robot description, xacro)
@@ -71,5 +71,5 @@
   <xacro:arg name="camera_far_clip" default="20.0"/>
   <xacro:arg name="camera_noise_mean" default="0.0"/>
-  <xacro:arg name="camera_noise_stddev" default="0.004"/>
+  <xacro:arg name="camera_noise_stddev" default="0.003"/>
   <xacro:arg name="camera_visualize" default="false"/>
   <xacro:arg name="inspection_led_x" default="0.380"/>

File: src/climbot_gazebo/worlds/climbot_wall.sdf.xacro (robot description, xacro)
@@ -30,8 +30,12 @@
   <xacro:arg name="ambient_g" default="0.025"/>
   <xacro:arg name="ambient_b" default="0.025"/>
-  <xacro:arg name="environment_intensity" default="0.035"/>
-  <xacro:arg name="environment_direction_x" default="-1.0"/>
-  <xacro:arg name="environment_direction_y" default="0.2"/>
-  <xacro:arg name="environment_direction_z" default="-0.4"/>
+  <xacro:arg name="moonlight_intensity" default="0.30"/>
+  <xacro:arg name="moonlight_direction_x" default="-1.0"/>
+  <xacro:arg name="moonlight_direction_y" default="0.2"/>
+  <xacro:arg name="moonlight_direction_z" default="-0.4"/>
+  <xacro:arg name="moonlight_diffuse_r" default="0.85"/>
+  <xacro:arg name="moonlight_diffuse_g" default="0.88"/>
+  <xacro:arg name="moonlight_diffuse_b" default="0.95"/>
+  <xacro:arg name="moonlight_cast_shadows" default="true"/>
   <xacro:property name="centre_x" value="$(arg centre_x)"/>
   <xacro:property name="centre_y" value="$(arg centre_y)"/>
@@ -157,14 +161,41 @@
       </persistent>
     </plugin>
-    <!-- Weak night environment only. It intentionally casts no shadow: the
-         inspection LED on the robot is the dominant, measured illuminant. -->
-    <light type="directional" name="night_environment">
-      <cast_shadows>false</cast_shadows>
+    <!-- One physical moonlight, weaker than the robot LED but with real
+         directional shadows. It is a scene light, not a GUI-only override. -->
+    <light type="directional" name="moonlight">
+      <cast_shadows>$(arg moonlight_cast_shadows)</cast_shadows>
       <pose>4 -2 8 0 0 0</pose>
-      <diffuse>1 1 1 1</diffuse>
+      <diffuse>$(arg moonlight_diffuse_r) $(arg moonlight_diffuse_g) $(arg moonlight_diffuse_b) 1</diffuse>
       <specular>0.02 0.02 0.02 1</specular>
-      <intensity>$(arg environment_intensity)</intensity>
-      <direction>$(arg environment_direction_x) $(arg environment_direction_y) $(arg environment_direction_z)</direction>
+      <intensity>$(arg moonlight_intensity)</intensity>
+      <direction>$(arg moonlight_direction_x) $(arg moonlight_direction_y) $(arg moonlight_direction_z)</direction>
     </light>
+    <!-- A physical reference for the operator's perspective.  Its top sits
+         20 mm below work y = 0, so it cannot perturb wheel/wall contact at
+         the wall foot while still catching a falling robot. -->
+    <model name="ground">
+      <static>true</static>
+      <pose>0 0 -0.02 0 0 0</pose>
+      <link name="ground_link">
+        <collision name="ground_collision">
+          <geometry>
+            <plane><normal>0 0 1</normal><size>30 30</size></plane>
+          </geometry>
+          <surface>
+            <friction><ode><mu>0.8</mu><mu2>0.8</mu2></ode></friction>
+          </surface>
+        </collision>
+        <visual name="ground_visual">
+          <geometry>
+            <plane><normal>0 0 1</normal><size>30 30</size></plane>
+          </geometry>
+          <material>
+            <ambient>0.22 0.24 0.28 1</ambient>
+            <diffuse>0.38 0.42 0.48 1</diffuse>
+            <specular>0.02 0.02 0.02 1</specular>
+          </material>
+        </visual>
+      </link>
+    </model>
     <model name="wall">
       <static>true</static>
