Commit message: style: paint the chassis orange in both the URDF and the SDF
The chassis was blue and the small heading marker on its front edge was
orange. Swapping the body to orange would have made the marker vanish
into it, and that marker is the only cue for which way the robot faces in
RViz and in Gazebo screenshots of turns, so it goes dark instead.

The two descriptions carry the colour separately - RViz reads the URDF,
Gazebo the rendered SDF - so both are changed together and the SDF
ambient keeps the same 0.7 ratio to diffuse the blue used.

Co-Authored-By: Claude Opus 5 <noreply@anthropic.com>

File: src/climbot_description/urdf/climbot.urdf.xacro (robot description, xacro)
@@ -41,9 +41,12 @@
   <xacro:property name="caster_offset_x" value="$(arg caster_x)"/>
   <xacro:property name="caster_offset_z" value="${caster_radius}"/>
-  <material name="body_blue">
-    <color rgba="0.10 0.32 0.80 1"/>
+  <material name="body_orange">
+    <color rgba="0.95 0.45 0.05 1"/>
   </material>
-  <material name="marker_orange">
-    <color rgba="1.0 0.32 0.05 1"/>
+  <!-- The heading marker has to read against the chassis, so it turned dark
+       when the chassis turned orange. It is the only cue for which way the
+       robot faces in RViz and in Gazebo screenshots of turns. -->
+  <material name="marker_dark">
+    <color rgba="0.12 0.13 0.15 1"/>
   </material>
   <material name="wheel_black">
@@ -100,5 +103,5 @@
         <box size="${length} ${width} ${thickness}"/>
       </geometry>
-      <material name="body_blue"/>
+      <material name="body_orange"/>
     </visual>
     <visual>
@@ -108,5 +111,5 @@
         <box size="0.07 ${width * 0.41} 0.025"/>
       </geometry>
-      <material name="marker_orange"/>
+      <material name="marker_dark"/>
     </visual>
     <collision>

File: src/climbot_gazebo/models/climbot/model.sdf.xacro (robot description, xacro)
@@ -171,6 +171,6 @@
         </geometry>
         <material>
-          <ambient>0.08 0.22 0.55 1</ambient>
-          <diffuse>0.10 0.32 0.80 1</diffuse>
+          <ambient>0.66 0.31 0.03 1</ambient>
+          <diffuse>0.95 0.45 0.05 1</diffuse>
           <specular>0.25 0.25 0.25 1</specular>
         </material>
@@ -183,7 +183,9 @@
           </box>
         </geometry>
+        <!-- Dark, not orange: it has to stay readable against the orange
+             chassis. Matches marker_dark in climbot.urdf.xacro. -->
         <material>
-          <ambient>0.9 0.25 0.05 1</ambient>
-          <diffuse>1.0 0.32 0.05 1</diffuse>
+          <ambient>0.08 0.09 0.10 1</ambient>
+          <diffuse>0.12 0.13 0.15 1</diffuse>
         </material>
       </visual>

Commit message: fix: give the heading marker its own link so RViz paints it dark
Painting the chassis orange left the marker orange in RViz even though the
rendered URDF asks for marker_dark: RViz gives a link one material and
applies it to every visual on it, so the second visual on base_link
inherited the chassis colour. Gazebo honours per-visual materials and
already showed it dark.

Move the marker to a fixed-joint child link, which is per-link by
construction. It carries no inertia and only the URDF changes - Gazebo
spawns the SDF, where the marker stays a chassis visual and the physics
model gains nothing massless. Geometry and pose are identical in both, and
robot_state_publisher now emits front_marker_link on /tf_static.

Co-Authored-By: Claude Opus 5 <noreply@anthropic.com>

File: src/climbot_description/urdf/climbot.urdf.xacro (robot description, xacro)
@@ -105,12 +105,4 @@
       <material name="body_orange"/>
     </visual>
-    <visual>
-      <origin xyz="${base_x + length / 2.0 - 0.03} ${base_y}
-                   ${base_z + thickness / 2.0 + 0.011}"/>
-      <geometry>
-        <box size="0.07 ${width * 0.41} 0.025"/>
-      </geometry>
-      <material name="marker_dark"/>
-    </visual>
     <collision>
       <origin xyz="${base_x} ${base_y} ${base_z}"/>
@@ -120,4 +112,24 @@
     </collision>
   </link>
+  <!-- The heading marker is its own link only because RViz paints every
+       visual of a link with one material: as a second visual on base_link it
+       came out the same orange as the chassis and stopped showing which way
+       the robot faces. Gazebo does honour per-visual materials, so in
+       model.sdf.xacro it stays a visual on the chassis and no massless link
+       is added to the physics model. Geometry and pose are the same in both. -->
+  <link name="front_marker_link">
+    <visual>
+      <geometry>
+        <box size="0.07 ${width * 0.41} 0.025"/>
+      </geometry>
+      <material name="marker_dark"/>
+    </visual>
+  </link>
+  <joint name="front_marker_joint" type="fixed">
+    <parent link="base_link"/>
+    <child link="front_marker_link"/>
+    <origin xyz="${base_x + length / 2.0 - 0.03} ${base_y}
+                 ${base_z + thickness / 2.0 + 0.011}"/>
+  </joint>
   <!-- The IMU is co-located with base_link, so this frame is coincident
        with it. It exists so an offset mount only needs robot.yaml changed. -->
