Commit message: test: add asymmetric G1 camera target

File: src/climbot_gazebo/worlds/climbot_wall.sdf.xacro (robot description, xacro)
@@ -21,4 +21,9 @@
   <xacro:arg name="spawn_pitch" default="0.0"/>
   <xacro:arg name="spawn_yaw" default="1.5707963267948966"/>
+  <xacro:arg name="inspection_target" default="false"/>
+  <xacro:arg name="target_lateral" default="0.3"/>
+  <xacro:arg name="target_height" default="2.0"/>
+  <xacro:arg name="target_length" default="0.28125"/>
+  <xacro:arg name="target_width" default="0.5"/>
   <xacro:property name="centre_x" value="$(arg centre_x)"/>
   <xacro:property name="centre_y" value="$(arg centre_y)"/>
@@ -28,4 +33,8 @@
   <xacro:property name="height" value="$(arg height)"/>
   <xacro:property name="grid_spacing" value="$(arg grid_spacing)"/>
+  <xacro:property name="target_lateral" value="$(arg target_lateral)"/>
+  <xacro:property name="target_height" value="$(arg target_height)"/>
+  <xacro:property name="target_length" value="$(arg target_length)"/>
+  <xacro:property name="target_width" value="$(arg target_width)"/>
   <!-- Wall face, the plane the wheels roll on, and the grid overlay just
        in front of it so the decals never fight the collision surface. -->
@@ -157,4 +166,34 @@
           <xacro:grid_line axis="row" index="1" count="${rows}"/>
         </xacro:if>
+        <!-- Optional G1 acceptance target. Work +X (robot-forward at spawn)
+             is world +Y and must appear at image top; work +Y is world +Z
+             and must appear at image left. Red marks +X, green marks +Y.
+             It is off by default and never belongs in inspection imagery. -->
+        <xacro:if value="$(arg inspection_target)">
+          <visual name="g1_target_background">
+            <pose>${decal_x + 0.004} ${target_lateral} ${target_height - centre_z} 0 0 0</pose>
+            <geometry><box><size>0.004 ${target_length} ${target_width}</size></box></geometry>
+            <material>
+              <ambient>0.95 0.95 0.95 1</ambient>
+              <diffuse>0.95 0.95 0.95 1</diffuse>
+              <specular>0 0 0 1</specular>
+            </material>
+          </visual>
+          <visual name="g1_target_forward_red">
+            <pose>${decal_x + 0.007} ${target_lateral + 0.35 * target_length} ${target_height - centre_z} 0 0 0</pose>
+            <geometry><box><size>0.004 ${0.18 * target_length} ${0.10 * target_width}</size></box></geometry>
+            <material><ambient>1 0.02 0.02 1</ambient><diffuse>1 0.02 0.02 1</diffuse></material>
+          </visual>
+          <visual name="g1_target_up_green">
+            <pose>${decal_x + 0.007} ${target_lateral} ${target_height - centre_z + 0.35 * target_width} 0 0 0</pose>
+            <geometry><box><size>0.004 ${0.10 * target_length} ${0.18 * target_width}</size></box></geometry>
+            <material><ambient>0.02 1 0.02 1</ambient><diffuse>0.02 1 0.02 1</diffuse></material>
+          </visual>
+          <visual name="g1_target_centre_blue">
+            <pose>${decal_x + 0.007} ${target_lateral} ${target_height - centre_z} 0 0 0</pose>
+            <geometry><box><size>0.004 ${0.08 * target_length} ${0.08 * target_width}</size></box></geometry>
+            <material><ambient>0.02 0.02 1 1</ambient><diffuse>0.02 0.02 1 1</diffuse></material>
+          </visual>
+        </xacro:if>
       </link>
     </model>

Commit message: test: measure rectified camera line residual

File: src/climbot_gazebo/worlds/climbot_wall.sdf.xacro (robot description, xacro)
@@ -92,4 +92,25 @@
     </xacro:if>
   </xacro:macro>
+  <xacro:macro name="g1_target_line" params="axis index count">
+    <xacro:if value="${index &lt; count}">
+      <xacro:property name="fraction" value="${-0.4 + 0.8 * index / (count - 1)}"/>
+      <visual name="g1_target_grid_${axis}_${index}">
+        <xacro:if value="${axis == 'forward'}">
+          <pose>${decal_x + 0.0055} ${target_lateral + fraction * target_length} ${target_height - centre_z} 0 0 0</pose>
+          <geometry><box><size>0.003 ${0.010 * target_length} ${0.90 * target_width}</size></box></geometry>
+        </xacro:if>
+        <xacro:unless value="${axis == 'forward'}">
+          <pose>${decal_x + 0.0055} ${target_lateral} ${target_height - centre_z + fraction * target_width} 0 0 0</pose>
+          <geometry><box><size>0.003 ${0.90 * target_length} ${0.006 * target_width}</size></box></geometry>
+        </xacro:unless>
+        <material>
+          <ambient>1 1 0.01 1</ambient>
+          <diffuse>1 1 0.01 1</diffuse>
+          <specular>0 0 0 1</specular>
+        </material>
+      </visual>
+      <xacro:g1_target_line axis="${axis}" index="${index + 1}" count="${count}"/>
+    </xacro:if>
+  </xacro:macro>
   <world name="climbot_wall">
     <gravity>0 0 -9.81</gravity>
@@ -180,4 +201,6 @@
             </material>
           </visual>
+          <xacro:g1_target_line axis="forward" index="0" count="5"/>
+          <xacro:g1_target_line axis="cross" index="0" count="9"/>
           <visual name="g1_target_forward_red">
             <pose>${decal_x + 0.007} ${target_lateral + 0.35 * target_length} ${target_height - centre_z} 0 0 0</pose>

Commit message: test: verify inspection camera view clearance

File: src/climbot_gazebo/worlds/climbot_wall.sdf.xacro (robot description, xacro)
@@ -107,4 +107,5 @@
           <ambient>1 1 0.01 1</ambient>
           <diffuse>1 1 0.01 1</diffuse>
+          <emissive>1 1 0.01 1</emissive>
           <specular>0 0 0 1</specular>
         </material>
@@ -198,4 +199,5 @@
               <ambient>0.95 0.95 0.95 1</ambient>
               <diffuse>0.95 0.95 0.95 1</diffuse>
+              <emissive>0.95 0.95 0.95 1</emissive>
               <specular>0 0 0 1</specular>
             </material>
@@ -206,15 +208,15 @@
             <pose>${decal_x + 0.007} ${target_lateral + 0.35 * target_length} ${target_height - centre_z} 0 0 0</pose>
             <geometry><box><size>0.004 ${0.18 * target_length} ${0.10 * target_width}</size></box></geometry>
-            <material><ambient>1 0.02 0.02 1</ambient><diffuse>1 0.02 0.02 1</diffuse></material>
+            <material><ambient>1 0.02 0.02 1</ambient><diffuse>1 0.02 0.02 1</diffuse><emissive>1 0.02 0.02 1</emissive></material>
           </visual>
           <visual name="g1_target_up_green">
             <pose>${decal_x + 0.007} ${target_lateral} ${target_height - centre_z + 0.35 * target_width} 0 0 0</pose>
             <geometry><box><size>0.004 ${0.10 * target_length} ${0.18 * target_width}</size></box></geometry>
-            <material><ambient>0.02 1 0.02 1</ambient><diffuse>0.02 1 0.02 1</diffuse></material>
+            <material><ambient>0.02 1 0.02 1</ambient><diffuse>0.02 1 0.02 1</diffuse><emissive>0.02 1 0.02 1</emissive></material>
           </visual>
           <visual name="g1_target_centre_blue">
             <pose>${decal_x + 0.007} ${target_lateral} ${target_height - centre_z} 0 0 0</pose>
             <geometry><box><size>0.004 ${0.08 * target_length} ${0.08 * target_width}</size></box></geometry>
-            <material><ambient>0.02 0.02 1 1</ambient><diffuse>0.02 0.02 1 1</diffuse></material>
+            <material><ambient>0.02 0.02 1 1</ambient><diffuse>0.02 0.02 1 1</diffuse><emissive>0.02 0.02 1 1</emissive></material>
           </visual>
         </xacro:if>
