Commit message: refactor: generate the Gazebo world from the wall description
The world restated every wall dimension as a literal, so wall.yaml and
the SDF could disagree, and the sixteen grid decals were copy-pasted
blocks that had to be re-cut by hand for any other wall size.

Render the world from climbot_wall.sdf.xacro at launch time using
wall.yaml, deriving the slab, its friction, the reference grid, the
suction force and the robot spawn pose from that one description. The
grid is now generated for whatever wall size and spacing are configured.
The rendered document has the same 493-tag structure as the world it
replaces, and re-running the contact load measurement reproduces the
recorded baseline on every manoeuvre.

Also replaces the unconditional WSL environment variables with a
gpu_backend argument that defaults to detecting WSL, so the launch no
longer forces Mesa's D3D12 driver on machines with a native GPU.

Co-Authored-By: Claude Opus 5 <noreply@anthropic.com>

File: src/climbot_gazebo/worlds/climbot_wall.sdf.xacro (robot description, xacro)
@@ -1,4 +1,65 @@
 <?xml version="1.0"?>
-<sdf version="1.10">
+<!--
+  Rendered at launch time from config/wall.yaml, which is the single source
+  of truth for the wall slab and the wall work frame. Nothing here may
+  restate a wall dimension as a literal.
+-->
+<sdf version="1.10" xmlns:xacro="http://www.ros.org/wiki/xacro">
+  <xacro:arg name="centre_x" default="0.0"/>
+  <xacro:arg name="centre_y" default="0.0"/>
+  <xacro:arg name="centre_z" default="4.0"/>
+  <xacro:arg name="thickness" default="0.10"/>
+  <xacro:arg name="width" default="10.0"/>
+  <xacro:arg name="height" default="8.0"/>
+  <xacro:arg name="mu" default="1.1"/>
+  <xacro:arg name="grid_spacing" default="1.0"/>
+  <xacro:arg name="suction_force" default="220.0"/>
+  <xacro:arg name="spawn_gap" default="0.001"/>
+  <xacro:arg name="spawn_lateral" default="0.0"/>
+  <xacro:arg name="spawn_height" default="2.0"/>
+  <xacro:arg name="spawn_roll" default="1.5707963267948966"/>
+  <xacro:arg name="spawn_pitch" default="0.0"/>
+  <xacro:arg name="spawn_yaw" default="1.5707963267948966"/>
+  <xacro:property name="centre_x" value="$(arg centre_x)"/>
+  <xacro:property name="centre_y" value="$(arg centre_y)"/>
+  <xacro:property name="centre_z" value="$(arg centre_z)"/>
+  <xacro:property name="thickness" value="$(arg thickness)"/>
+  <xacro:property name="width" value="$(arg width)"/>
+  <xacro:property name="height" value="$(arg height)"/>
+  <xacro:property name="grid_spacing" value="$(arg grid_spacing)"/>
+  <!-- Wall face, the plane the wheels roll on, and the grid overlay just
+       in front of it so the decals never fight the collision surface. -->
+  <xacro:property name="face_x" value="${centre_x + thickness / 2.0}"/>
+  <xacro:property name="decal_x" value="${thickness / 2.0 + 0.003}"/>
+  <!-- Outermost grid line sits one spacing inside each edge. -->
+  <xacro:property name="columns" value="${int(width / (2.0 * grid_spacing)) - 1}"/>
+  <xacro:property name="rows" value="${int(height / (2.0 * grid_spacing)) - 1}"/>
+  <xacro:macro name="grid_line" params="axis index count">
+    <xacro:if value="${index &lt;= 2 * count}">
+      <visual name="grid_${axis}_${index}">
+        <xacro:if value="${axis == 'column'}">
+          <pose>${decal_x} ${(index - count) * grid_spacing} 0 0 0 0</pose>
+          <geometry>
+            <box>
+              <size>0.006 ${0.035 if index == count else 0.025} ${height}</size>
+            </box>
+          </geometry>
+        </xacro:if>
+        <xacro:unless value="${axis == 'column'}">
+          <pose>${decal_x} 0 ${(index - count) * grid_spacing} 0 0 0</pose>
+          <geometry>
+            <box>
+              <size>0.006 ${width} ${0.035 if index == count else 0.025}</size>
+            </box>
+          </geometry>
+        </xacro:unless>
+        <material>
+          <ambient>${'0.10 0.12 0.16' if index == count else '0.18 0.20 0.24'} 1</ambient>
+          <diffuse>${'0.10 0.12 0.16' if index == count else '0.18 0.20 0.24'} 1</diffuse>
+        </material>
+      </visual>
+      <xacro:grid_line axis="${axis}" index="${index + 1}" count="${count}"/>
+    </xacro:if>
+  </xacro:macro>
   <world name="climbot_wall">
     <gravity>0 0 -9.81</gravity>
@@ -27,5 +88,6 @@
         <entity_name>climbot</entity_name>
         <entity_type>model</entity_type>
-        <force>-220 0 0</force>
+        <!-- Along the inward wall normal, which is world -X for this wall. -->
+        <force>${-1.0 * float("$(arg suction_force)")} 0 0</force>
         <torque>0 0 0</torque>
       </persistent>
@@ -41,9 +103,9 @@
       <static>true</static>
       <link name="wall_link">
-        <pose>0 0 4 0 0 0</pose>
+        <pose>${centre_x} ${centre_y} ${centre_z} 0 0 0</pose>
         <collision name="wall_collision">
           <geometry>
             <box>
-              <size>0.10 10.0 8.0</size>
+              <size>${thickness} ${width} ${height}</size>
             </box>
           </geometry>
@@ -51,6 +113,6 @@
             <friction>
               <ode>
-                <mu>1.1</mu>
-                <mu2>1.1</mu2>
+                <mu>$(arg mu)</mu>
+                <mu2>$(arg mu)</mu2>
               </ode>
             </friction>
@@ -60,5 +122,5 @@
           <geometry>
             <box>
-              <size>0.10 10.0 8.0</size>
+              <size>${thickness} ${width} ${height}</size>
             </box>
           </geometry>
@@ -69,91 +131,15 @@
           </material>
         </visual>
-        <!-- High-contrast one-metre grid on the 10 m x 8 m wall front face. -->
-        <visual name="grid_vertical_m4">
-          <pose>0.053 -4 0 0 0 0</pose>
-          <geometry><box><size>0.006 0.025 8.0</size></box></geometry>
-          <material><ambient>0.18 0.20 0.24 1</ambient><diffuse>0.18 0.20 0.24 1</diffuse></material>
-        </visual>
-        <visual name="grid_vertical_m3">
-          <pose>0.053 -3 0 0 0 0</pose>
-          <geometry><box><size>0.006 0.025 8.0</size></box></geometry>
-          <material><ambient>0.18 0.20 0.24 1</ambient><diffuse>0.18 0.20 0.24 1</diffuse></material>
-        </visual>
-        <visual name="grid_vertical_m2">
-          <pose>0.053 -2 0 0 0 0</pose>
-          <geometry><box><size>0.006 0.025 8.0</size></box></geometry>
-          <material><ambient>0.18 0.20 0.24 1</ambient><diffuse>0.18 0.20 0.24 1</diffuse></material>
-        </visual>
-        <visual name="grid_vertical_m1">
-          <pose>0.053 -1 0 0 0 0</pose>
-          <geometry><box><size>0.006 0.025 8.0</size></box></geometry>
-          <material><ambient>0.18 0.20 0.24 1</ambient><diffuse>0.18 0.20 0.24 1</diffuse></material>
-        </visual>
-        <visual name="grid_vertical_0">
-          <pose>0.053 0 0 0 0 0</pose>
-          <geometry><box><size>0.006 0.035 8.0</size></box></geometry>
-          <material><ambient>0.10 0.12 0.16 1</ambient><diffuse>0.10 0.12 0.16 1</diffuse></material>
-        </visual>
-        <visual name="grid_vertical_p1">
-          <pose>0.053 1 0 0 0 0</pose>
-          <geometry><box><size>0.006 0.025 8.0</size></box></geometry>
-          <material><ambient>0.18 0.20 0.24 1</ambient><diffuse>0.18 0.20 0.24 1</diffuse></material>
-        </visual>
-        <visual name="grid_vertical_p2">
-          <pose>0.053 2 0 0 0 0</pose>
-          <geometry><box><size>0.006 0.025 8.0</size></box></geometry>
-          <material><ambient>0.18 0.20 0.24 1</ambient><diffuse>0.18 0.20 0.24 1</diffuse></material>
-        </visual>
-        <visual name="grid_vertical_p3">
-          <pose>0.053 3 0 0 0 0</pose>
-          <geometry><box><size>0.006 0.025 8.0</size></box></geometry>
-          <material><ambient>0.18 0.20 0.24 1</ambient><diffuse>0.18 0.20 0.24 1</diffuse></material>
-        </visual>
-        <visual name="grid_vertical_p4">
-          <pose>0.053 4 0 0 0 0</pose>
-          <geometry><box><size>0.006 0.025 8.0</size></box></geometry>
-          <material><ambient>0.18 0.20 0.24 1</ambient><diffuse>0.18 0.20 0.24 1</diffuse></material>
-        </visual>
-        <visual name="grid_horizontal_m3">
-          <pose>0.053 0 -3 0 0 0</pose>
-          <geometry><box><size>0.006 10.0 0.025</size></box></geometry>
-          <material><ambient>0.18 0.20 0.24 1</ambient><diffuse>0.18 0.20 0.24 1</diffuse></material>
-        </visual>
-        <visual name="grid_horizontal_m2">
-          <pose>0.053 0 -2 0 0 0</pose>
-          <geometry><box><size>0.006 10.0 0.025</size></box></geometry>
-          <material><ambient>0.18 0.20 0.24 1</ambient><diffuse>0.18 0.20 0.24 1</diffuse></material>
-        </visual>
-        <visual name="grid_horizontal_m1">
-          <pose>0.053 0 -1 0 0 0</pose>
-          <geometry><box><size>0.006 10.0 0.025</size></box></geometry>
-          <material><ambient>0.18 0.20 0.24 1</ambient><diffuse>0.18 0.20 0.24 1</diffuse></material>
-        </visual>
-        <visual name="grid_horizontal_0">
-          <pose>0.053 0 0 0 0 0</pose>
-          <geometry><box><size>0.006 10.0 0.035</size></box></geometry>
-          <material><ambient>0.10 0.12 0.16 1</ambient><diffuse>0.10 0.12 0.16 1</diffuse></material>
-        </visual>
-        <visual name="grid_horizontal_p1">
-          <pose>0.053 0 1 0 0 0</pose>
-          <geometry><box><size>0.006 10.0 0.025</size></box></geometry>
-          <material><ambient>0.18 0.20 0.24 1</ambient><diffuse>0.18 0.20 0.24 1</diffuse></material>
-        </visual>
-        <visual name="grid_horizontal_p2">
-          <pose>0.053 0 2 0 0 0</pose>
-          <geometry><box><size>0.006 10.0 0.025</size></box></geometry>
-          <material><ambient>0.18 0.20 0.24 1</ambient><diffuse>0.18 0.20 0.24 1</diffuse></material>
-        </visual>
-        <visual name="grid_horizontal_p3">
-          <pose>0.053 0 3 0 0 0</pose>
-          <geometry><box><size>0.006 10.0 0.025</size></box></geometry>
-          <material><ambient>0.18 0.20 0.24 1</ambient><diffuse>0.18 0.20 0.24 1</diffuse></material>
-        </visual>
+        <!-- High-contrast reference grid on the wall front face. -->
+        <xacro:grid_line axis="column" index="0" count="${columns}"/>
+        <xacro:grid_line axis="row" index="0" count="${rows}"/>
       </link>
     </model>
     <include>
       <uri>model://climbot</uri>
-      <!-- local +X -> world +Y, local +Y -> world +Z, local +Z -> world +X -->
-      <pose>0.051 0 2.0 1.57079632679 0 1.57079632679</pose>
+      <!-- On the wall face, oriented so the robot's axes match the wall
+           work frame: local +X -> wall +X, +Y -> wall +Y, +Z -> wall normal. -->
+      <pose>${face_x + float("$(arg spawn_gap)")} $(arg spawn_lateral) $(arg spawn_height)
+            $(arg spawn_roll) $(arg spawn_pitch) $(arg spawn_yaw)</pose>
     </include>
     <gui fullscreen="false">
@@ -169,5 +155,5 @@
         <background_color>0.12 0.14 0.18</background_color>
         <!-- Front-on view centred on the robot's initial pose. -->
-        <camera_pose>2.8 0 2.0 0 0 3.14159265359</camera_pose>
+        <camera_pose>${face_x + 2.75} $(arg spawn_lateral) $(arg spawn_height) 0 0 3.14159265359</camera_pose>
       </plugin>
       <plugin filename="EntityContextMenuPlugin" name="Entity context menu">

Commit message: feat: make the wall reference grid switchable, in Gazebo and live in RViz
The grid has to go for runs that photograph the wall: it is a periodic
high-contrast pattern standing 3 mm proud of the surface, and at the
0.50 by 0.28 m photo footprint it lands in 67% of the images. It is worth
keeping for a human watching a plan. So it becomes a switch rather than a
decision: wall_grid_spacing:=0 removes it from both views for a whole run,
and the RViz display can be unticked live without restarting anything.

Three things had to be fixed to make one switch mean one grid.

The two views were not drawing the same lines. Gazebo spaced them one
pitch in from each edge, a rule written when the work frame's origin was
the wall's centre. Both now use whole multiples of the pitch measured from
the origin, interior lines only. The default 10 x 8 m wall at 1 m renders
identically - columns 1..9, rows 1..7, heavier line at x=5 and y=4 - so
docs/images/gazebo_wall.png stays valid.

coverage.rviz carried an rviz_default_plugins/Grid, which draws a square
centred on the fixed frame. That was right until the origin moved to the
corner and left a 10 x 10 m square hanging off it. It is now a MarkerArray
on /coverage/wall_grid, cut to the wall, latched and published once.

The pitch lived in simulation.yaml, which RViz cannot read. It moves to
wall.yaml as reference_grid.spacing_m, behind wall_frame's
reference_grid_spacing(), so all four launch files read one number.

test_coverage_wall_grid_off.py covers the off case, and the node test now
compares line coordinates rather than counting them; it was checked to
fail when the start index is moved back to 0.

Co-Authored-By: Claude Opus 5 <noreply@anthropic.com>

File: src/climbot_gazebo/worlds/climbot_wall.sdf.xacro (robot description, xacro)
@@ -32,29 +32,50 @@
   <xacro:property name="face_x" value="${centre_x + thickness / 2.0}"/>
   <xacro:property name="decal_x" value="${thickness / 2.0 + 0.003}"/>
-  <!-- Outermost grid line sits one spacing inside each edge. -->
-  <xacro:property name="columns" value="${int(width / (2.0 * grid_spacing)) - 1}"/>
-  <xacro:property name="rows" value="${int(height / (2.0 * grid_spacing)) - 1}"/>
+  <!-- Lines sit at whole multiples of the spacing measured from the work
+       frame's origin, the wall's lower-left corner, so a line is a work
+       coordinate an operator can read off the wall. Only the interior ones are
+       drawn: a line on an edge would hang half off the wall. RViz draws the
+       same lines from the same rule over /coverage/wall_grid, and both take
+       the spacing from climbot_description/config/wall.yaml.
+       A non-positive spacing removes the grid entirely. It is a periodic
+       high-contrast pattern standing 3 mm proud of the wall face, which puts
+       it in 67% of inspection photographs at the 0.50 m by 0.28 m footprint
+       those are taken at. Runs that photograph the wall switch it off, because
+       a repeating feature is what makes a stitch match the wrong place
+       confidently, and one that is not coplanar with the surface breaks the
+       homography the stitch assumes. Runs a human watches keep it. -->
+  <xacro:property name="show_grid" value="${grid_spacing > 0.0}"/>
+  <!-- The epsilon keeps a line off the far edge when the span divides exactly,
+       which is the ordinary case: 10 m at 1 m pitch is nine lines, not ten. -->
+  <xacro:property name="columns"
+                  value="${int((width - 1e-9) / grid_spacing) if show_grid else 0}"/>
+  <xacro:property name="rows"
+                  value="${int((height - 1e-9) / grid_spacing) if show_grid else 0}"/>
+  <!-- index counts lines from the work origin, so index * grid_spacing is the
+       line's work coordinate. The pose is relative to the link centre, hence
+       the half-span subtracted. The mid-span line is drawn heavier, which is
+       what makes the grid readable as two halves rather than as stripes. -->
   <xacro:macro name="grid_line" params="axis index count">
-    <xacro:if value="${index &lt;= 2 * count}">
+    <xacro:if value="${index &lt;= count}">
       <visual name="grid_${axis}_${index}">
         <xacro:if value="${axis == 'column'}">
-          <pose>${decal_x} ${(index - count) * grid_spacing} 0 0 0 0</pose>
-          <geometry>
-            <box>
-              <size>0.006 ${0.035 if index == count else 0.025} ${height}</size>
+          <pose>${decal_x} ${index * grid_spacing - width / 2.0} 0 0 0 0</pose>
+          <geometry>
+            <box>
+              <size>0.006 ${0.035 if fabs(index * grid_spacing - width / 2.0) &lt; 1e-9 else 0.025} ${height}</size>
             </box>
           </geometry>
         </xacro:if>
         <xacro:unless value="${axis == 'column'}">
-          <pose>${decal_x} 0 ${(index - count) * grid_spacing} 0 0 0</pose>
-          <geometry>
-            <box>
-              <size>0.006 ${width} ${0.035 if index == count else 0.025}</size>
+          <pose>${decal_x} 0 ${index * grid_spacing - height / 2.0} 0 0 0</pose>
+          <geometry>
+            <box>
+              <size>0.006 ${width} ${0.035 if fabs(index * grid_spacing - height / 2.0) &lt; 1e-9 else 0.025}</size>
             </box>
           </geometry>
         </xacro:unless>
         <material>
-          <ambient>${'0.10 0.12 0.16' if index == count else '0.18 0.20 0.24'} 1</ambient>
-          <diffuse>${'0.10 0.12 0.16' if index == count else '0.18 0.20 0.24'} 1</diffuse>
+          <ambient>${'0.10 0.12 0.16' if fabs(index * grid_spacing - (width if axis == 'column' else height) / 2.0) &lt; 1e-9 else '0.18 0.20 0.24'} 1</ambient>
+          <diffuse>${'0.10 0.12 0.16' if fabs(index * grid_spacing - (width if axis == 'column' else height) / 2.0) &lt; 1e-9 else '0.18 0.20 0.24'} 1</diffuse>
         </material>
       </visual>
@@ -132,6 +153,8 @@
         </visual>
         <!-- High-contrast reference grid on the wall front face. -->
-        <xacro:grid_line axis="column" index="0" count="${columns}"/>
-        <xacro:grid_line axis="row" index="0" count="${rows}"/>
+        <xacro:if value="${show_grid}">
+          <xacro:grid_line axis="column" index="1" count="${columns}"/>
+          <xacro:grid_line axis="row" index="1" count="${rows}"/>
+        </xacro:if>
       </link>
     </model>

Commit message: Photograph the plane the wheels ride on
The texture blocks stood 1.25 mm in front of the wall's collision face:
SURFACE_OFFSET_M lifted them 1 mm to keep the renderer from choosing
between two coplanar surfaces, and half the block's own 0.5 mm thickness
added the rest. The wheels rode on the collision face while the camera
photographed a film floating above it, which no real wall does.

At the 0.275 m camera distance that standoff makes the true object
distance 0.27375 m, so every mosaic came out scaled by +4566 ppm -- 43 mm
across a 9.5 m wall. It arrived as an absolute anchor offset that pose
optimisation cannot remove, because the images agree with each other
perfectly at the wrong scale; the error is isotropic, which is what ruled
out the two independently calibrated focal lengths as the cause.

Measured on the P2-06 joint mosaic by reprojecting the same 1340 frames
onto z = 0.00125 m: scale error 4590 -> 25 ppm, absolute anchor offset
P95 20.62 -> 1.20 mm, local residual P95 0.921 -> 0.245 mm. The pose-only
variant barely moved, as expected of a variant dominated by localisation
noise rather than projection geometry.

Blocks now put their outer face on the collision face and wall_visual is
recessed behind it, so nothing is coplanar and the mosaic's default
wall_plane_z_m of zero is the plane that was actually photographed. The
grid lines and the G1 target still sit 3 mm proud; they are not
photogrammetry inputs, but the same arithmetic applies to anything that
becomes one.

Co-Authored-By: Claude Opus 5 <noreply@anthropic.com>
Claude-Session: https://claude.ai/code/session_01CEyov6A2fjGw3vcPPeBouV

File: src/climbot_gazebo/worlds/climbot_wall.sdf.xacro (robot description, xacro)
@@ -53,4 +53,6 @@
   <xacro:property name="face_x" value="${centre_x + thickness / 2.0}"/>
   <xacro:property name="decal_x" value="${thickness / 2.0 + 0.003}"/>
+  <!-- How far wall_visual sits behind the collision face; see wall_visual. -->
+  <xacro:property name="wall_visual_recess" value="0.001"/>
   <!-- Lines sit at whole multiples of the spacing measured from the work
        frame's origin, the wall's lower-left corner, so a line is a work
@@ -217,8 +219,14 @@
           </surface>
         </collision>
+        <!-- Recessed behind the collision face. Texture blocks put their
+             outer face exactly on that face, because the camera must
+             photograph the plane the wheels ride on; a coplanar wall_visual
+             would then z-fight with every block. Nothing measures this
+             surface, so moving it back costs only a 1 mm step visible at the
+             texture border under grazing light. -->
         <visual name="wall_visual">
           <geometry>
             <box>
-              <size>${thickness} ${width} ${height}</size>
+              <size>${thickness - 2.0 * wall_visual_recess} ${width} ${height}</size>
             </box>
           </geometry>
