Commit message: Take the P2-06 acceptance domain out of the evidence chain
The coverage gate asked whether every feature pixel inside a region was
photographed, and that region arrived as four numbers on a command line.
Whoever ran the checker therefore chose what the run would be judged
against, and several ways of choosing badly ended in a pass: a NaN vertex
compares false against every pixel, a region outside the mosaic selects
none, and both left the gate reporting that nothing uncovered had been
found inside nothing. The region now comes out of the evidence --

    mosaic manifest -> processed runs -> source archives -> frozen task

-- with every link checked by digest, so naming the wrong run is refused
rather than answered. The archives already carried the task snapshot; it
had simply never been read. A region with no feature pixels in it is now
an error, not a pass.

It is a polygon, not a bounding box, because the planner already accepts
trapezoid tasks whose bounding box would accept ground the task excludes.
And it is called the inspection region, not the reachable one: the camera
footprint is carried 0.340 m ahead of the robot centre and reaches
0.481 m past a boundary the centre may not cross, so pixels outside the
region are not thereby unphotographable. Saying they were stated as
physics what is only a choice of acceptance domain. The summary now
splits them by an observable envelope instead, and only the pixels
outside it are described as out of reach.

The other half is provenance. A formal summary was filed naming commit
ec62a54 with source_modified false, for fields produced by code that did
not exist until 139a21e -- a claim no program could have made, and none
had: it was typed. Every mosaic stage now publishes its own record next
to its own products, inside the same atomic rename, and the summary
generator reads the chain and checks that each stage read what the stage
before it wrote. climbot_common exists so that git_state, which was
built to prevent exactly this and which the entire mosaic chain had
skipped, can be called without dragging rclpy into a package that only
wants numpy; its third copy, one field short and one pathspec narrow,
has been merged into it. tools is now inside the default pathspec,
because that is where the generator runs from.

Also: wall_visual only steps back from the collision face when texture
blocks are loaded to z-fight with it. Unconditionally recessed, it put
the plain wall's visible surface 1 mm behind the plane the wheels ride
on -- the same class of error, reversed, as the blocks that once stood
1.25 mm proud of it and scaled every mosaic by +4566 ppm.

And the fusion memory budget says what it is: a soft budget for planning
parallelism, not a limit on process memory. It warns when it cannot buy
a worker instead of returning 1 in silence, and does not refuse, because
its fixed cost was fitted on the largest mosaic here and a small job
would be turned away for memory it never uses.

Co-Authored-By: Claude Opus 5 <noreply@anthropic.com>
Claude-Session: https://claude.ai/code/session_01CEyov6A2fjGw3vcPPeBouV

File: src/climbot_gazebo/worlds/climbot_wall.sdf.xacro (robot description, xacro)
@@ -53,6 +53,12 @@
   <xacro:property name="face_x" value="${centre_x + thickness / 2.0}"/>
   <xacro:property name="decal_x" value="${thickness / 2.0 + 0.003}"/>
-  <!-- How far wall_visual sits behind the collision face; see wall_visual. -->
-  <xacro:property name="wall_visual_recess" value="0.001"/>
+  <!-- How far wall_visual sits behind the collision face, and only when it
+       has to be: the recess exists to stop texture blocks z-fighting with a
+       coplanar wall face, so without those blocks it does nothing but move the
+       visible surface 1 mm off the plane the wheels ride on. That is the same
+       kind of error, in the opposite direction, as the one that scaled every
+       mosaic by +4566 ppm, so it is not left switched on by default. -->
+  <xacro:property name="wall_visual_recess"
+                 value="${0.001 if '$(arg inspection_target)' in ('true', 'True', '1') else 0.0}"/>
   <!-- Lines sit at whole multiples of the spacing measured from the work
        frame's origin, the wall's lower-left corner, so a line is a work
